File: hardware/interface.kicad_sch (KiCad schematic)
At the start: 0 parts

Commit message: hw: Add USB Type-C interface
Parts:
- added USB?: HRO-TYPE-C-31-M-12, Type-C:HRO-TYPE-C-31-M-12-HandSoldering, symbol Type-C:HRO-TYPE-C-31-M-12
Connections:
- new net GND: USB?.1 (GND), USB?.12 (GND), USB?.13 (SHIELD)
- new net USB_DM: USB?.7 (DN1)
- new net USB_DP: USB?.6 (DP1)
- new net VBUS: USB?.11 (VBUS), USB?.2 (VBUS)
- no-connect marks 0 -> 6
Changed lines of the file:
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@@
 (kicad_sch (version 20211123) (generator eeschema)
   (paper "A4")
+  (junction (at 85.09 92.71) (diameter 0) (color 0 0 0 0)
+  )
+  (junction (at 85.09 95.25) (diameter 0) (color 0 0 0 0)
+  )
+  (no_connect (at 81.28 82.55))
+  (no_connect (at 81.28 85.09))
+  (no_connect (at 81.28 74.93))
+  (no_connect (at 81.28 87.63))
+  (no_connect (at 81.28 72.39))
+  (no_connect (at 81.28 69.85))
+  (wire (pts (xy 81.28 67.31) (xy 88.9 67.31))
+    (stroke (width 0) (type default) (color 0 0 0 0))
+  )
+  (wire (pts (xy 193.04 74.93) (xy 216.535 74.93))
+    (stroke (width 0) (type default) (color 0 0 0 0))
+  )
+  (wire (pts (xy 81.28 80.01) (xy 97.155 80.01))
+    (stroke (width 0) (type default) (color 0 0 0 0))
+  )
+  (wire (pts (xy 81.28 95.25) (xy 85.09 95.25))
+    (stroke (width 0) (type default) (color 0 0 0 0))
+  )
+  (wire (pts (xy 81.28 77.47) (xy 97.155 77.47))
+    (stroke (width 0) (type default) (color 0 0 0 0))
+  )
+  (wire (pts (xy 193.04 77.47) (xy 216.535 77.47))
+    (stroke (width 0) (type default) (color 0 0 0 0))
+  )
+  (wire (pts (xy 81.28 64.77) (xy 85.09 64.77))
+    (stroke (width 0) (type default) (color 0 0 0 0))
+  )
+  (wire (pts (xy 81.28 90.17) (xy 88.9 90.17))
+    (stroke (width 0) (type default) (color 0 0 0 0))
+  )
+  (wire (pts (xy 85.09 95.25) (xy 85.09 99.06))
+    (stroke (width 0) (type default) (color 0 0 0 0))
+  )
+  (wire (pts (xy 88.9 95.25) (xy 85.09 95.25))
+    (stroke (width 0) (type default) (color 0 0 0 0))
+  )
+  (wire (pts (xy 85.09 92.71) (xy 85.09 95.25))
+    (stroke (width 0) (type default) (color 0 0 0 0))
+  )
+  (wire (pts (xy 81.28 92.71) (xy 85.09 92.71))
+    (stroke (width 0) (type default) (color 0 0 0 0))
+  )
+  (wire (pts (xy 85.09 64.77) (xy 85.09 92.71))
+    (stroke (width 0) (type default) (color 0 0 0 0))
+  )
+  (label "USB_DP" (at 97.155 77.47 180)
+    (effects (font (size 1.27 1.27)) (justify right bottom))
+  )
+  (label "USB_DM" (at 193.04 77.47 0)
+    (effects (font (size 1.27 1.27)) (justify left bottom))
+  )
+  (label "USB_DP" (at 193.04 74.93 0)
+    (effects (font (size 1.27 1.27)) (justify left bottom))
+  )
+  (label "USB_DM" (at 97.155 80.01 180)
+    (effects (font (size 1.27 1.27)) (justify right bottom))
+  )
+  (hierarchical_label "USB_DM" (shape bidirectional) (at 216.535 77.47 0)
+    (effects (font (size 1.27 1.27)) (justify left))
+  )
+  (hierarchical_label "USB_DP" (shape bidirectional) (at 216.535 74.93 0)
+    (effects (font (size 1.27 1.27)) (justify left))
+  )
+  (symbol (lib_id "power:GND") (at 85.09 99.06 0) (unit 1)
+    (in_bom yes) (on_board yes)
+    (property "Reference" "#PWR?" (id 0) (at 85.09 105.41 0)
+      (effects (font (size 1.27 1.27)) hide)
+    )
+    (property "Value" "GND" (id 1) (at 85.217 103.4542 0)
+      (effects (font (size 1.27 1.27)) hide)
+    )
+    (property "Footprint" "" (id 2) (at 85.09 99.06 0)
+      (effects (font (size 1.27 1.27)) hide)
+    )
+    (property "Datasheet" "" (id 3) (at 85.09 99.06 0)
+      (effects (font (size 1.27 1.27)) hide)
+    )
+    (pin "1")
+  )
+  (symbol (lib_id "power:PWR_FLAG") (at 88.9 95.25 270) (unit 1)
+    (in_bom yes) (on_board yes)
+    (property "Reference" "#FLG?" (id 0) (at 90.805 95.25 0)
+      (effects (font (size 1.27 1.27)) hide)
+    )
+    (property "Value" "PWR_FLAG" (id 1) (at 92.1512 95.25 90)
+      (effects (font (size 1.27 1.27)) (justify left) hide)
+    )
+    (property "Footprint" "" (id 2) (at 88.9 95.25 0)
+      (effects (font (size 1.27 1.27)) hide)
+    )
+    (property "Datasheet" "~" (id 3) (at 88.9 95.25 0)
+      (effects (font (size 1.27 1.27)) hide)
+    )
+    (pin "1")
+  )
+  (symbol (lib_id "power:VBUS") (at 88.9 90.17 270) (unit 1)
+    (in_bom yes) (on_board yes)
+    (property "Reference" "#PWR?" (id 0) (at 85.09 90.17 0)
+      (effects (font (size 1.27 1.27)) hide)
+    )
+    (property "Value" "VBUS" (id 1) (at 92.075 90.17 90)
+      (effects (font (size 1.27 1.27)) (justify left))
+    )
+    (property "Footprint" "" (id 2) (at 88.9 90.17 0)
+      (effects (font (size 1.27 1.27)) hide)
+    )
+    (property "Datasheet" "" (id 3) (at 88.9 90.17 0)
+      (effects (font (size 1.27 1.27)) hide)
+    )
+    (pin "1")
+  )
+  (symbol (lib_id "power:VBUS") (at 88.9 67.31 270) (unit 1)
+    (in_bom yes) (on_board yes)
+    (property "Reference" "#PWR?" (id 0) (at 85.09 67.31 0)
+      (effects (font (size 1.27 1.27)) hide)
+    )
+    (property "Value" "VBUS" (id 1) (at 92.075 67.31 90)
+      (effects (font (size 1.27 1.27)) (justify left))
+    )
+    (property "Footprint" "" (id 2) (at 88.9 67.31 0)
+      (effects (font (size 1.27 1.27)) hide)
+    )
+    (property "Datasheet" "" (id 3) (at 88.9 67.31 0)
+      (effects (font (size 1.27 1.27)) hide)
+    )
+    (pin "1")
+  )
+  (symbol (lib_id "Type-C:HRO-TYPE-C-31-M-12") (at 78.74 78.74 0) (unit 1)
+    (in_bom yes) (on_board yes)
+    (property "Reference" "USB?" (id 0) (at 74.4982 58.4962 0)
+      (effects (font (size 1.524 1.524)))
+    )
+    (property "Value" "HRO-TYPE-C-31-M-12" (id 1) (at 74.4982 61.1886 0)
+      (effects (font (size 1.524 1.524)))
+    )
+    (property "Footprint" "Type-C:HRO-TYPE-C-31-M-12-HandSoldering" (id 2) (at 78.74 78.74 0)
+      (effects (font (size 1.524 1.524)) hide)
+    )
+    (property "Datasheet" "" (id 3) (at 78.74 78.74 0)
+      (effects (font (size 1.524 1.524)) hide)
+    )
+    (property "LCSC" "C165948" (id 4) (at 78.74 78.74 0)
+      (effects (font (size 1.27 1.27)) hide)
+    )
+    (pin "1")
+    (pin "10")
+    (pin "11")
+    (pin "12")
+    (pin "13")
+    (pin "2")
+    (pin "3")
+    (pin "4")
+    (pin "5")
+    (pin "6")
+    (pin "7")
+    (pin "8")
+    (pin "9")
+  )
 )
